Commit message: irobot urdf model created

File: gazebo/iRobot.gazebo.xacro (robot description, xacro)
@@ -37,5 +37,5 @@
         <odometryTopic>odom</odometryTopic>
         <odometryFrame>odom</odometryFrame>
-        <odometrySource>world</odometrySource>
+        <odometrySource>encoder</odometrySource>
         <robotBaseFrame>base_link</robotBaseFrame>
         <updateRate>10.0</updateRate>

File: model/hokuyo.urdf.xacro (robot description, xacro)
@@ -2,56 +2,57 @@
 <robot xmlns:xacro="http://www.ros.org/wiki/xacro" name="hokuyo">
 <xacro:macro name="hokuyo_laser" params="xyz rpy parent">
-	  <joint name="hokuyo_laser_joint" type="fixed">
-		<axis xyz="0 0 1" />
-		<origin xyz="${xyz}" rpy="${rpy}"/>
-		<parent link="${parent}"/>
-		<child link="hokuyo_laser_link"/>
-	  </joint>
-	  <link name="hokuyo_laser_link">
-		<collision>
-		  <origin xyz="0 0 0" rpy="0 0 0"/>
-		  <geometry>
-			<box size="0.1 0.1 0.1"/>
-		  </geometry>
-		</collision>
-		<visual>
-		  <origin xyz="0 0 0" rpy="0 0 0"/>
-		  <geometry>
-            <cylinder length="0.1" radius="0.045"/>
-		  </geometry>
-		</visual>
-		<inertial>
-		  <mass value="1e-5" />
-		  <origin xyz="0 0 0" rpy="0 0 0"/>
-		  <inertia ixx="1e-6" ixy="0" ixz="0" iyy="1e-6" iyz="0" izz="1e-6" />
-		</inertial>
-	  </link>
-	  <gazebo reference="hokuyo_laser_link">
-		  <sensor type="ray" name="head_hokuyo_sensor">
-		  <pose>0 0 0 0 0 0</pose>
-          <visualize>true</visualize>
-          <update_rate>40</update_rate>
-			<ray>
-			  <scan>
-				<horizontal>
-				  <samples>720</samples>
-                  <resolution>1</resolution>
-                  <min_angle>-1.570796</min_angle>
-                  <max_angle>1.570796</max_angle>
-				</horizontal>
-			  </scan>
-			  <range>
-				<min>0.08</min>
-				<max>5</max>
-				<resolution>0.01</resolution>
-			  </range>
-			</ray>
-			<plugin name="gazebo_ros_head_hokuyo_controller" filename="libgazebo_ros_laser.so">
+    <joint name="hokuyo_laser_joint" type="fixed">
+        <axis xyz="0 0 1" />
+        <origin xyz="${xyz}" rpy="${rpy}"/>
+        <parent link="${parent}"/>
+        <child link="hokuyo_laser_link"/>
+    </joint>
+    <link name="hokuyo_laser_link">
+        <collision>
+            <origin xyz="0 0 0" rpy="0 0 0"/>
+            <geometry>
+                <box size="0.1 0.1 0.1"/>
+            </geometry>
+        </collision>
+        <visual>
+            <origin xyz="0 0 0" rpy="0 0 0"/>
+            <geometry>
+                <cylinder length="0.1" radius="0.045"/>
+            </geometry>
+        </visual>
+        <inertial>
+            <mass value="1e-5" />
+            <origin xyz="0 0 0" rpy="0 0 0"/>
+            <inertia ixx="1e-6" ixy="0" ixz="0" iyy="1e-6" iyz="0" izz="1e-6" />
+        </inertial>
+    </link>
+    <gazebo reference="hokuyo_laser_link">
+        <gravity>true</gravity>
+        <sensor type="ray" name="head_hokuyo_sensor">
+            <pose>0 0 0 0 0 0</pose>
+            <visualize>true</visualize>
+            <update_rate>40</update_rate>
+            <ray>
+                <scan>
+                    <horizontal>
+                        <samples>720</samples>
+                        <resolution>1</resolution>
+                        <min_angle>-1.570796</min_angle>
+                        <max_angle>1.570796</max_angle>
+                    </horizontal>
+                </scan>
+                <range>
+                    <min>0.08</min>
+                    <max>5</max>
+                    <resolution>0.01</resolution>
+                </range>
+            </ray>
+            <plugin name="gazebo_ros_head_hokuyo_controller" filename="libgazebo_ros_laser.so">
                 <robotNamespace></robotNamespace>
                 <topicName>laser_scan</topicName>
                 <frameName>hokuyo_laser_link</frameName>
-			</plugin>
-		  </sensor>
-	  </gazebo>
-  </xacro:macro>
+            </plugin>
+        </sensor>
+    </gazebo>
+</xacro:macro>
 </robot>

File: model/iRobot.urdf.xacro (robot description, xacro)
@@ -5,4 +5,5 @@
   <xacro:include filename="$(find irobotcreate2)/model/axis.urdf.xacro"/>
   <xacro:include filename="$(find irobotcreate2)/model/wheel.urdf.xacro"/>
+  <xacro:include filename="$(find irobotcreate2)/model/shelf.urdf.xacro"/>
   <xacro:include filename="$(find irobotcreate2)/gazebo/iRobot.gazebo.xacro"/>
   <xacro:include filename="$(find irobotcreate2)/model/hokuyo.urdf.xacro"/>
@@ -91,5 +92,5 @@
         </collision>
     </link>
-    <joint name="sphere_to_ground" type="fixed">
+<!--    <joint name="sphere_to_ground" type="fixed">
         <origin xyz="0 0 -0.03" rpy="0 0 0"/>
         <parent link="sphere"/>
@@ -102,5 +103,5 @@
             <inertia ixx="0.0" ixy="0.0" ixz="0.0" iyy="0.0" iyz="0.0" izz="0.0"/>
         </inertial>
-    </link>
+    </link>-->
     <joint name="base_front_joint" type="fixed">
         <origin xyz="0.14 0 0.04" rpy="0 0 0"/>
@@ -132,4 +133,13 @@
                   parent="base_link">
     </xacro:hokuyo_laser>
+  <!--  <xacro:model_shelf name="first_shelf"
+                       parent="chassis"
+                       height="0.15">
+    </xacro:model_shelf>
+    <xacro:model_shelf name="second_shelf"
+                       parent="first_shelf"
+                       height="0.25">
+    </xacro:model_shelf>
+    -->
     <xacro:iRobot_gazebo />
 </robot>

Commit message: create new launch files

File: gazebo/iRobot.gazebo.xacro (robot description, xacro)
@@ -6,5 +6,16 @@
     <gazebo reference="ground">
     </gazebo>
-    <gazebo reference="sphere">
+    <gazebo reference="sphere1">
+      <gravity>true</gravity>
+      <material>Gazebo/Grey</material>
+      <mu1>0</mu1>
+      <mu2>0</mu2>
+      <kp>10000000</kp>
+      <kd>1</kd>
+      <fdir1>1 0 0</fdir1>
+      <minDepth>0.0001</minDepth>
+      <maxContacts>1</maxContacts>
+    </gazebo>
+    <gazebo reference="sphere2">
       <gravity>true</gravity>
       <material>Gazebo/Grey</material>
@@ -30,6 +41,6 @@
         <leftJoint>left_wheel_rot_joint</leftJoint>
         <rightJoint>right_wheel_rot_joint</rightJoint>
-        <wheelSeparation>0.32</wheelSeparation>
-        <wheelDiameter>0.14</wheelDiameter>
+        <wheelSeparation>0.28</wheelSeparation>
+        <wheelDiameter>0.06</wheelDiameter>
         <torque>20</torque>
         <wheelAcceleration>1.8</wheelAcceleration>
