Commit message: broken gazebo urdfs fixed, gazebo should now be able to run

File: model/axis.urdf.xacro (robot description, xacro)
@@ -14,6 +14,6 @@
                 <origin xyz="0 0 0" rpy="${-pi/2} 0 0"/>
                 <mass value="${small_mass}"/>
-                <inertia ixx="${1/12*small_mass*3*0.0025^2+1/12*small_mass*0.02^2)}" ixy="0.0" ixz="0.0" iyy="${1/12*small_mass*3*0.0025^2+1/12*small_mass*0.02^2)}" iyz="0.0"
-                                izz="${1/12*small_mass*0.0025^2}"/>
+                <inertia ixx="${1/12*small_mass*3*0.0025**2+1/12*small_mass*0.02**2}" ixy="0.0" ixz="0.0" iyy="${1/12*small_mass*3*0.0025**2+1/12*small_mass*0.02**2}" iyz="0.0"
+                                izz="${1/12*small_mass*0.0025**2}"/>
             </inertial>
         <visual>

File: model/iRobot.urdf.xacro (robot description, xacro)
@@ -29,5 +29,5 @@
             <origin xyz="0 0 0" rpy="0 0 0"/>
             <mass value="10"/>
-             <inertia ixx="${1/12*10*3*0.17^2+1/12*5*3*0.08^2}" ixy="0.0" ixz="0.0" iyy="${1/12*10*3*0.17^2+1/12*5*3*0.08^2}" iyz="0.0" izz="${1/2*10*0.17^2}"/>
+             <inertia ixx="${1/12*10*3*0.17**2+1/12*5*3*0.08**2}" ixy="0.0" ixz="0.0" iyy="${1/12*10*3*0.17**2+1/12*5*3*0.08**2}" iyz="0.0" izz="${1/2*10*0.17**2}"/>
         </inertial>
         <visual>
@@ -78,5 +78,5 @@
             <origin xyz="0 0 0" rpy="0 0 0"/>
             <mass value="${sphere_mass}"/>
-            <inertia ixx="${2/5*sphere_mass*0.01^2}" ixy="0.0" ixz="0.0" iyy="${2/5*sphere_mass*0.01^2}" iyz="0.0" izz="${2/5*sphere_mass*0.01^2}"/>
+            <inertia ixx="${2/5*sphere_mass*0.01**2}" ixy="0.0" ixz="0.0" iyy="${2/5*sphere_mass*0.01**2}" iyz="0.0" izz="${2/5*sphere_mass*0.01**2}"/>
         </inertial>
         <visual>
@@ -105,5 +105,5 @@
             <origin xyz="0 0 0" rpy="0 0 0"/>
             <mass value="${sphere_mass}"/>
-            <inertia ixx="${2/5*sphere_mass*0.01^2}" ixy="0.0" ixz="0.0" iyy="${2/5*sphere_mass*0.01^2}" iyz="0.0" izz="${2/5*sphere_mass*0.01^2}"/>
+            <inertia ixx="${2/5*sphere_mass*0.01**2}" ixy="0.0" ixz="0.0" iyy="${2/5*sphere_mass*0.01**2}" iyz="0.0" izz="${2/5*sphere_mass*0.01**2}"/>
         </inertial>
         <visual>

File: model/wheel.urdf.xacro (robot description, xacro)
@@ -16,5 +16,5 @@
             <origin xyz="0 0.01 0" rpy="${-pi/2} 0 0"/>
             <mass value="${mass}"/>
-            <inertia ixx="${1/12*mass*3*radius^2+1/12*mass*width^2)}" ixy="0.0" ixz="0.0" iyy="${1/12*mass*3*radius^2+1/12*mass*width^2)}" iyz="0.0" izz="${1/12*mass*radius^2}"/>
+            <inertia ixx="${1/12*mass*3*radius**2+1/12*mass*width**2}" ixy="0.0" ixz="0.0" iyy="${1/12*mass*3*radius**2+1/12*mass*width**2}" iyz="0.0" izz="${1/12*mass*radius**2}"/>
         </inertial>
         <visual>
