Commit message: fixed parameters in diff_drive plugin and added a second sphere in the irobot model

File: iRobot/iRobot.urdf (robot description, URDF)
Before this commit: robot iRobot, 9 links, 8 joints
Links:
- removed link sphere
- added link sphere1, mass 0.3; collision sphere radius=0.01; visual sphere radius=0.01
- added link sphere2, mass 0.3; collision sphere radius=0.01; visual sphere radius=0.01
- link hokuyo_laser_link: geometry collision cylinder length=0.05 radius=0.045; visual cylinder length=0.05 radius=0.045
Joints:
- removed joint sphere_joint
- added joint sphere_joint1: type revolute, parent chassis, child sphere1, origin xyz=0.14 0 -0.04 rpy=0 0 0, axis 0 0 1, limit lower=0 upper=0 effort=100 velocity=100
- added joint sphere_joint2: type revolute, parent chassis, child sphere2, origin xyz=-0.14 0 -0.04 rpy=0 0 0, axis 0 0 1, limit lower=0 upper=0 effort=100 velocity=100
- joint hokuyo_laser_joint: origin xyz=0 0 0.05 rpy=0 0 0 -> xyz=0 0 0.065 rpy=0 0 0; parent base_link -> chassis
- joint left_axis_base_joint: origin xyz=-0.04 0.14 -0.02 rpy=0 0 0 -> xyz=0 0.14 -0.02 rpy=0 0 0
- joint right_axis_base_joint: origin xyz=-0.04 -0.14 -0.02 rpy=0 0 0 -> xyz=0 -0.14 -0.02 rpy=0 0 0

File: model/hokuyo.urdf.xacro (robot description, xacro)
@@ -12,5 +12,5 @@
             <origin xyz="0 0 0" rpy="0 0 0"/>
             <geometry>
-                <box size="0.1 0.1 0.1"/>
+                <cylinder length="0.05" radius="0.045"/>
             </geometry>
         </collision>
@@ -18,5 +18,5 @@
             <origin xyz="0 0 0" rpy="0 0 0"/>
             <geometry>
-                <cylinder length="0.1" radius="0.045"/>
+                <cylinder length="0.05" radius="0.045"/>
             </geometry>
         </visual>

File: model/iRobot.urdf.xacro (robot description, xacro)
@@ -45,5 +45,5 @@
     <xacro:model_axis name="left_axis"
                       parent="chassis">
-    <origin xyz="-0.04 0.14 -0.02" rpy="0 0 0"/>
+    <origin xyz="0 0.14 -0.02" rpy="0 0 0"/>
     </xacro:model_axis>
    <xacro:model_wheel name="left_wheel"
@@ -56,5 +56,5 @@
     <xacro:model_axis name="right_axis"
                       parent="chassis">
-    <origin xyz="-0.04 -0.14 -0.02" rpy="0 0 0"/>
+    <origin xyz="0 -0.14 -0.02" rpy="0 0 0"/>
     </xacro:model_axis>
     <xacro:model_wheel name="right_wheel"
@@ -65,12 +65,39 @@
     <origin xyz="0 0 0" rpy="0 0 0"/>
     </xacro:model_wheel>
-    <joint name="sphere_joint" type="revolute">
+    <joint name="sphere_joint1" type="revolute">
         <origin xyz="0.14 0 -0.04" rpy="0 0 0"/>
         <axis xyz="0 0 1"/>
         <limit lower="0" upper="0" effort="100" velocity="100"/>
         <parent link="chassis"/>
-        <child link="sphere"/>
+        <child link="sphere1"/>
     </joint>
-    <link name="sphere">
+    <link name="sphere1">
+        <inertial>
+            <origin xyz="0 0 0" rpy="0 0 0"/>
+            <mass value="${sphere_mass}"/>
+            <inertia ixx="${2/5*sphere_mass*0.01^2}" ixy="0.0" ixz="0.0" iyy="${2/5*sphere_mass*0.01^2}" iyz="0.0" izz="${2/5*sphere_mass*0.01^2}"/>
+        </inertial>
+        <visual>
+            <origin xyz="0 0 0" rpy="0 0 0"/>
+            <geometry>
+                <sphere radius="0.01"/>
+            </geometry>
+            <material name="iRobot/Grey"/>
+        </visual>
+        <collision>
+            <origin xyz="0 0 0" rpy="0 0 0"/>
+            <geometry>
+                <sphere radius="0.01"/>
+            </geometry>
+        </collision>
+    </link>
+    <joint name="sphere_joint2" type="revolute">
+        <origin xyz="-0.14 0 -0.04" rpy="0 0 0"/>
+        <axis xyz="0 0 1"/>
+        <limit lower="0" upper="0" effort="100" velocity="100"/>
+        <parent link="chassis"/>
+        <child link="sphere2"/>
+    </joint>
+    <link name="sphere2">
         <inertial>
             <origin xyz="0 0 0" rpy="0 0 0"/>
@@ -129,9 +156,10 @@
         </collision>
     </link>
-    <xacro:hokuyo_laser xyz="0 0 0.05"
+    <!-- Laser position: x y 0.025(laser height)+parent_height -->
+    <xacro:hokuyo_laser xyz="0 0 ${0.025+0.04}"
                   rpy="0 0 0"
-                  parent="base_link">
+                  parent="chassis">
     </xacro:hokuyo_laser>
-  <!--  <xacro:model_shelf name="first_shelf"
+<!--    <xacro:model_shelf name="first_shelf"
                        parent="chassis"
                        height="0.15">
@@ -140,6 +168,5 @@
                        parent="first_shelf"
                        height="0.25">
-    </xacro:model_shelf>
-    -->
+    </xacro:model_shelf>-->
     <xacro:iRobot_gazebo />
 </robot>

Commit message: update models

File: iRobot/iRobot.urdf (robot description, URDF)
Before this commit: robot iRobot, 10 links, 9 joints
Links:
- removed link hokuyo_laser_link
- added link laser_link, mass 1e-5; collision cylinder length=0.05 radius=0.045; visual cylinder length=0.05 radius=0.045
Joints:
- joint hokuyo_laser_joint: child hokuyo_laser_link -> laser_link

File: model/hokuyo.urdf.xacro (robot description, xacro)
@@ -6,7 +6,7 @@
         <origin xyz="${xyz}" rpy="${rpy}"/>
         <parent link="${parent}"/>
-        <child link="hokuyo_laser_link"/>
+        <child link="laser_link"/>
     </joint>
-    <link name="hokuyo_laser_link">
+    <link name="laser_link">
         <collision>
             <origin xyz="0 0 0" rpy="0 0 0"/>
@@ -27,7 +27,7 @@
         </inertial>
     </link>
-    <gazebo reference="hokuyo_laser_link">
+    <gazebo reference="laser_link">
         <gravity>true</gravity>
-        <sensor type="ray" name="head_hokuyo_sensor">
+        <sensor type="ray" name="head_sensor">
             <pose>0 0 0 0 0 0</pose>
             <visualize>true</visualize>
@@ -38,6 +38,6 @@
                         <samples>720</samples>
                         <resolution>1</resolution>
-                        <min_angle>-1.570796</min_angle>
-                        <max_angle>1.570796</max_angle>
+                        <min_angle>-3.14159</min_angle>
+                        <max_angle>3.14159</max_angle>
                     </horizontal>
                 </scan>
@@ -47,9 +47,18 @@
                     <resolution>0.01</resolution>
                 </range>
+                <noise>
+                    <type>gaussian</type>
+                    <!-- Noise parameters based on published spec for Hokuyo laser
+                        achieving "+-30mm" accuracy at range < 10m.  A mean of 0.0m and
+                        stddev of 0.01m will put 99.7% of samples within 0.03m of the true
+                        reading. -->
+                    <mean>0.0</mean>
+                    <stddev>0.001</stddev>
+                </noise>
             </ray>
             <plugin name="gazebo_ros_head_hokuyo_controller" filename="libgazebo_ros_laser.so">
                 <robotNamespace></robotNamespace>
                 <topicName>laser_scan</topicName>
-                <frameName>hokuyo_laser_link</frameName>
+                <frameName>laser_link</frameName>
             </plugin>
         </sensor>

Commit message: using new imu plugin

File: iRobot/iRobot.urdf (robot description, URDF)
Before this commit: robot iRobot, 9 links, 8 joints
Links:
- added link imu_sensor_link, mass 1e-5; collision box size=0.03 0.03 0.03; visual box size=0.03 0.03 0.03
Joints:
- added joint imu_sensor_joint: type fixed, parent base_link, child imu_sensor_link, origin xyz=-0.1 0 0.05 rpy=0 0 0, axis 0 0 1

File: model/iRobot.urdf.xacro (robot description, xacro)
@@ -8,4 +8,5 @@
   <xacro:include filename="$(find irobotcreate2)/gazebo/iRobot.gazebo.xacro"/>
   <xacro:include filename="$(find irobotcreate2)/model/hokuyo.urdf.xacro"/>
+  <xacro:include filename="$(find irobotcreate2)/model/imu.urdf.xacro"/>
   <xacro:property name="pi" value="3.1415926535897931"/>
   <xacro:property name="wheel_mass" value="0.5"/>
@@ -133,4 +134,8 @@
                   parent="base_link">
     </xacro:hokuyo_laser>
+    <xacro:imu_sensor xyz="-0.1 0 0.05"
+                  rpy="0 0 0"
+                  parent="base_link">
+    </xacro:imu_sensor>
   <!--  <xacro:model_shelf name="first_shelf"
                        parent="chassis"

Commit message: fixed imu xacro

File: iRobot/iRobot.urdf (robot description, URDF)
Before this commit: robot iRobot, 10 links, 9 joints
Links:
- link imu_sensor_link: mass 1e-5 -> 0.001

File: model/imu.urdf.xacro (robot description, xacro)
@@ -20,15 +20,10 @@
                 <box size="0.03 0.03 0.03"/>
             </geometry>
-	    <material>
-		<script>
-		    <name>Gazebo/Red</name>
-		    <uri>__default__</uri>
-		</script>
-	    </material>
+            <material name="iRobot/Red"/>
         </visual>
         <inertial>
-            <mass value="1e-5" />
+            <mass value="0.001" />
             <origin xyz="0 0 0" rpy="0 0 0"/>
-            <inertia ixx="1e-6" ixy="0" ixz="0" iyy="1e-6" iyz="0" izz="1e-6" />
+            <inertia ixx="0.00000015" ixy="0" ixz="0" iyy="0.00000015" iyz="0" izz="0.00000015" />
         </inertial>
     </link>

Commit message: removed world and launch file

File: iRobot/iRobot.urdf (robot description, URDF)
Before this commit: robot iRobot, 10 links, 9 joints
Links:
- removed link front_marker
- removed link laser_link
- added link camera_link, mass 0.0001; collision box size=0.02 0.08 0.05; visual box size=0.02 0.08 0.05
- added link hokuyo_laser_link, mass 1e-5; collision cylinder length=0.04 radius=0.045; visual cylinder length=0.04 radius=0.045
- added link imu_sensor_link, mass 0.001; collision box size=0.02 0.02 0.02; visual box size=0.02 0.02 0.02
Joints:
- removed joint base_front_joint
- added joint camera_sensor_joint: type fixed, parent base_link, child camera_link, origin xyz=0 0 0.1 rpy=0 0 0, axis 0 1 0
- added joint imu_sensor_joint: type fixed, parent base_link, child imu_sensor_link, origin xyz=-0.1 0 0.05 rpy=0 0 0, axis 0 0 1
- joint hokuyo_laser_joint: child laser_link -> hokuyo_laser_link; origin xyz=0 0 0.065 rpy=0 0 0 -> xyz=0 0 0.06 rpy=0 0 0; parent chassis -> base_link

File: model/axis.urdf.xacro (robot description, xacro)
@@ -1,35 +1,35 @@
 <?xml version="1.0"?>
 <robot xmlns:xacro="http://www.ros.org/wiki/xacro" name="axis">
- <xacro:include filename="$(find irobotcreate2)/gazebo/axis.gazebo.xacro"/>
-<xacro:property name="pi" value="3.1415926535897931"/>
-<xacro:property name="small_mass" value="0.001"/>
-<xacro:macro name="model_axis" params="name parent *origin">
-    <joint name="${name}_base_joint" type="fixed">
-	<insert_block name="origin"/>
-        <parent link="${parent}"/>
-        <child link="${name}"/>
-    </joint>
-    <link name="${name}">
-        <inertial>
+    <xacro:include filename="$(find irobotcreate2)/gazebo/axis.gazebo.xacro"/>
+    <xacro:property name="pi" value="3.1415926535897931"/>
+    <xacro:property name="small_mass" value="0.001"/>
+    <xacro:macro name="model_axis" params="name parent *origin">
+        <joint name="${name}_base_joint" type="fixed">
+            <insert_block name="origin"/>
+            <parent link="${parent}"/>
+            <child link="${name}"/>
+        </joint>
+        <link name="${name}">
+            <inertial>
+                <origin xyz="0 0 0" rpy="${-pi/2} 0 0"/>
+                <mass value="${small_mass}"/>
+                <inertia ixx="${1/12*small_mass*3*0.0025^2+1/12*small_mass*0.02^2)}" ixy="0.0" ixz="0.0" iyy="${1/12*small_mass*3*0.0025^2+1/12*small_mass*0.02^2)}" iyz="0.0"
+                                izz="${1/12*small_mass*0.0025^2}"/>
+            </inertial>
+        <visual>
             <origin xyz="0 0 0" rpy="${-pi/2} 0 0"/>
-            <mass value="${small_mass}"/>
-            <inertia ixx="${1/12*small_mass*3*0.0025^2+1/12*small_mass*0.02^2)}" ixy="0.0" ixz="0.0" iyy="${1/12*small_mass*3*0.0025^2+1/12*small_mass*0.02^2)}" iyz="0.0"
-izz="${1/12*small_mass*0.0025^2}"/>
-        </inertial>
-	<visual>
-	    <origin xyz="0 0 0" rpy="${-pi/2} 0 0"/>
-	    <geometry>
-            <cylinder length="0.02" radius="0.0025"/>
-	    </geometry>
-	    <material name="iRobot/Red"/>
-	</visual>
-	<collision>
-	    <origin xyz="0 0 0" rpy="${-pi/2} 0 0"/>
-	    <geometry>
-            <cylinder length="0.02" radius="0.0025"/>
-	    </geometry>
-        </collision>
-    </link>
-    <xacro:axis_gazebo name="${name}"/>
-</xacro:macro>
+            <geometry>
+                <cylinder length="0.02" radius="0.0025"/>
+            </geometry>
+            <material name="iRobot/MediumGray"/>
+        </visual>
+        <collision>
+            <origin xyz="0 0 0" rpy="${-pi/2} 0 0"/>
+            <geometry>
+                <cylinder length="0.02" radius="0.0025"/>
+            </geometry>
+            </collision>
+        </link>
+        <xacro:axis_gazebo name="${name}"/>
+    </xacro:macro>
 </robot>

File: model/hokuyo.urdf.xacro (robot description, xacro)
@@ -6,11 +6,11 @@
         <origin xyz="${xyz}" rpy="${rpy}"/>
         <parent link="${parent}"/>
-        <child link="laser_link"/>
+        <child link="hokuyo_laser_link"/>
     </joint>
-    <link name="laser_link">
+    <link name="hokuyo_laser_link">
         <collision>
             <origin xyz="0 0 0" rpy="0 0 0"/>
             <geometry>
-                <cylinder length="0.05" radius="0.045"/>
+                <cylinder length="0.04" radius="0.045"/>
             </geometry>
         </collision>
@@ -18,6 +18,7 @@
             <origin xyz="0 0 0" rpy="0 0 0"/>
             <geometry>
-                <cylinder length="0.05" radius="0.045"/>
+                <cylinder length="0.04" radius="0.045"/>
             </geometry>
+            <material name="iRobot/LightBlue"/>
         </visual>
         <inertial>
@@ -27,7 +28,7 @@
         </inertial>
     </link>
-    <gazebo reference="laser_link">
+    <gazebo reference="hokuyo_laser_link">
         <gravity>true</gravity>
-        <sensor type="ray" name="head_sensor">
+        <sensor type="ray" name="head_hokuyo_sensor">
             <pose>0 0 0 0 0 0</pose>
             <visualize>true</visualize>
@@ -56,5 +57,5 @@
                 <robotNamespace></robotNamespace>
                 <topicName>laser_scan</topicName>
-                <frameName>laser_link</frameName>
+                <frameName>hokuyo_laser_link</frameName>
             </plugin>
         </sensor>

File: model/iRobot.urdf.xacro (robot description, xacro)
@@ -8,4 +8,6 @@
   <xacro:include filename="$(find irobotcreate2)/gazebo/iRobot.gazebo.xacro"/>
   <xacro:include filename="$(find irobotcreate2)/model/hokuyo.urdf.xacro"/>
+  <xacro:include filename="$(find irobotcreate2)/model/imu.urdf.xacro"/>
+  <xacro:include filename="$(find irobotcreate2)/model/camera.urdf.xacro"/>
   <xacro:property name="pi" value="3.1415926535897931"/>
   <xacro:property name="wheel_mass" value="0.5"/>
@@ -34,5 +36,5 @@
                 <cylinder length="0.08" radius="0.17"/>
             </geometry>
-            <material name="iRobot/LightYellow"/>
+            <material name="iRobot/LightGrey"/>
         </visual>
         <collision>
@@ -83,5 +85,5 @@
                 <sphere radius="0.01"/>
             </geometry>
-            <material name="iRobot/Grey"/>
+            <material name="iRobot/Black"/>
         </visual>
         <collision>
@@ -110,5 +112,5 @@
                 <sphere radius="0.01"/>
             </geometry>
-            <material name="iRobot/Grey"/>
+            <material name="iRobot/Black"/>
         </visual>
         <collision>
@@ -119,54 +121,28 @@
         </collision>
     </link>
-<!--    <joint name="sphere_to_ground" type="fixed">
-        <origin xyz="0 0 -0.03" rpy="0 0 0"/>
-        <parent link="sphere"/>
-        <child link="ground"/>
-    </joint>
-    <link name="ground">
-        <inertial>
-            <origin xyz="0 0 0" rpy="0 0 0"/>
-            <mass value="0"/>
-            <inertia ixx="0.0" ixy="0.0" ixz="0.0" iyy="0.0" iyz="0.0" izz="0.0"/>
-        </inertial>
-    </link>-->
-    <joint name="base_front_joint" type="fixed">
-        <origin xyz="0.14 0 0.04" rpy="0 0 0"/>
-        <parent link="chassis"/>
-        <child link="front_marker"/>
-    </joint>
-    <link name="front_marker">
-        <inertial>
-            <origin xyz="0 0 0" rpy="0 0 0"/>
-            <mass value="0.001"/>
-            <inertia ixx="0.00001" ixy="0.0" ixz="0.0" iyy="0.00001" iyz="0.0" izz="0.00001"/>
-        </inertial>
-        <visual>
-            <origin xyz="0 0 0" rpy="0 0 0"/>
-            <geometry>
-                <cylinder length="0.01" radius="0.01"/>
-            </geometry>
-            <material name="iRobot/LightYellow"/>
-        </visual>
-        <collision>
-            <origin xyz="0 0 0" rpy="0 0 0"/>
-            <geometry>
-                <cylinder length="0.01" radius="0.01"/>
-            </geometry>
-        </collision>
-    </link>
-    <!-- Laser position: x y 0.025(laser height)+parent_height -->
-    <xacro:hokuyo_laser xyz="0 0 ${0.025+0.04}"
+    <!-- Laser link and plugin -->
+    <xacro:hokuyo_laser xyz="0 0 ${0.04 + 0.02}"
                   rpy="0 0 0"
-                  parent="chassis">
+                  parent="base_link">
     </xacro:hokuyo_laser>
+    <!--Imu link and plugin-->
+    <xacro:imu_sensor xyz="-0.1 0 ${0.04 + 0.01}"
+                  rpy="0 0 0"
+                  parent="base_link">
+    </xacro:imu_sensor>
+    <!--Camera link and plugin-->
+    <xacro:camera_sensor xyz="0 0 ${0.04 + 0.02 + 0.04}"
+                  rpy="0 0 0"
+                  parent="base_link">
+    </xacro:camera_sensor>
 <!--    <xacro:model_shelf name="first_shelf"
                        parent="chassis"
                        height="0.15">
-    </xacro:model_shelf>
-    <xacro:model_shelf name="second_shelf"
+    </xacro:model_shelf>-->
+<!--    <xacro:model_shelf name="second_shelf"
                        parent="first_shelf"
                        height="0.25">
-    </xacro:model_shelf>-->
+    </xacro:model_shelf>
+    -->
     <xacro:iRobot_gazebo />
 </robot>

File: model/wheel.urdf.xacro (robot description, xacro)
@@ -23,5 +23,5 @@
                 <cylinder length="${width}" radius="${radius}"/>
             </geometry>
-            <material name="iRobot/Grey"/>
+            <material name="iRobot/Black"/>
         </visual>
         <collision>

Commit message: partially working gmapping

File: iRobot/iRobot.urdf (robot description, URDF)
Before this commit: robot iRobot, 11 links, 10 joints
Links:
- added link dummy
Joints:
- added joint dummy_joint: type fixed, parent dummy, child base_link
